Commit message: fix color for gazebo7

File: hir_description/urdf/wheel/wheel.gazebo.xacro (robot description, xacro)
@@ -11,4 +11,7 @@
     <material>Gazebo/Orange</material>
   </gazebo>
+  <gazebo reference="visual_right_wheel">
+    <material>Gazebo/Orange</material>
+  </gazebo>
   <!-- Right Wheel -->
   <gazebo reference="right_wheel">
@@ -21,3 +24,6 @@
     <material>Gazebo/Orange</material>
   </gazebo>
+  <gazebo reference="visual_left_wheel">
+    <material>Gazebo/Orange</material>
+  </gazebo>
 </robot>

File: hir_description/urdf/wheel/wheel.urdf.xacro (robot description, xacro)
@@ -2,5 +2,5 @@
 <robot>
   <link name="visual_left_wheel">
-    <visual name="visual">
+    <visual>
       <origin xyz="0 0.03 0" rpy="0 3.1415 1.5707"/>
       <geometry>
@@ -23,5 +23,5 @@
   </link>
   <link name="visual_right_wheel">
-    <visual name="visual">
+    <visual>
       <origin xyz="0 -0.03 0" rpy="0 0 1.5707"/>
       <geometry>
