Commit message: modification to match gazebo

File: hir_description/urdf/base/base.urdf.xacro (robot description, xacro)
@@ -29,5 +29,5 @@
 		<origin xyz="-0.185 -0.0875 0.05" rpy="0 1.5707 1.5707" />
 		<geometry>
-			<cylinder length="0.03" radius="0.0485" />
+			<cylinder length="0.03" radius="0.04973" />
 		</geometry>
 	</collision>
@@ -35,5 +35,5 @@
 		<origin xyz="-0.185 0.0875 0.05" rpy="0 1.5707 1.5707" />
 		<geometry>
-			<cylinder length="0.03" radius="0.0487" />
+			<cylinder length="0.03" radius="0.04973" />
 		</geometry>
 	</collision>
@@ -41,5 +41,5 @@
 		<origin xyz="0.18 -0.0875 0.05" rpy="0 1.5707 1.5707" />
 		<geometry>
-			<cylinder length="0.03" radius="0.0487" />
+			<cylinder length="0.03" radius="0.04973" />
 		</geometry>
 	</collision>
@@ -47,5 +47,5 @@
 		<origin xyz="0.18 0.0875 0.05" rpy="0 1.5707 1.5707" />
 		<geometry>
-			<cylinder length="0.03" radius="0.0487" />
+			<cylinder length="0.03" radius="0.04973" />
 		</geometry>
 	</collision>
