Commit message: reduce file size

File: hir_description/urdf/manipulator/manipulator.transmission.xacro (robot description, xacro)
@@ -1,4 +1,16 @@
 <?xml version="1.0"?>
-<robot>
+<robot xmlns:xacro="http://www.ros.org/wiki/xacro">
+  <xacro:macro name="arm_transmission" params="name">
+	<transmission name="trans_${name}">
+	  <type>transmission_interface/SimpleTransmission</type>
+      <joint name="${name}_joint">
+        <hardwareInterface>EffortJointInterface</hardwareInterface>
+      </joint>
+      <actuator name="motor_{name}">
+        <hardwareInterface>EffortJointInterface</hardwareInterface>
+        <mechanicalReduction>1</mechanicalReduction>
+      </actuator>
+	</transmission>
+  </xacro:macro>
   <transmission name="trans_shoulder_slider">
     <type>transmission_interface/SimpleTransmission</type>
@@ -11,63 +23,9 @@
     </actuator>
   </transmission>
-  <transmission name="trans_shoulder_roll">
-    <type>transmission_interface/SimpleTransmission</type>
-    <joint name="shoulder_roll_joint">
-      <hardwareInterface>EffortJointInterface</hardwareInterface>
-    </joint>
-    <actuator name="motor_shoulder_roll">
-      <hardwareInterface>EffortJointInterface</hardwareInterface>
-      <mechanicalReduction>1</mechanicalReduction>
-    </actuator>
-  </transmission>
-  <transmission name="trans_shoulder_pitch">
-    <type>transmission_interface/SimpleTransmission</type>
-    <joint name="shoulder_pitch_joint">
-      <hardwareInterface>EffortJointInterface</hardwareInterface>
-    </joint>
-    <actuator name="motor_shoulder_pitch">
-      <hardwareInterface>EffortJointInterface</hardwareInterface>
-      <mechanicalReduction>1</mechanicalReduction>
-    </actuator>
-  </transmission>
-  <transmission name="trans_elbow_pitch">
-    <type>transmission_interface/SimpleTransmission</type>
-    <joint name="elbow_pitch_joint">
-      <hardwareInterface>EffortJointInterface</hardwareInterface>
-    </joint>
-    <actuator name="motor_elbow_pitch">
-      <hardwareInterface>EffortJointInterface</hardwareInterface>
-      <mechanicalReduction>1</mechanicalReduction>
-    </actuator>
-  </transmission>
-  <transmission name="trans_wrist_pitch">
-    <type>transmission_interface/SimpleTransmission</type>
-    <joint name="wrist_pitch_joint">
-      <hardwareInterface>EffortJointInterface</hardwareInterface>
-    </joint>
-    <actuator name="motor_wrist_pitch">
-      <hardwareInterface>EffortJointInterface</hardwareInterface>
-      <mechanicalReduction>1</mechanicalReduction>
-    </actuator>
-  </transmission>
-  <transmission name="trans_wrist_yaw">
-    <type>transmission_interface/SimpleTransmission</type>
-    <joint name="wrist_yaw_joint">
-      <hardwareInterface>EffortJointInterface</hardwareInterface>
-    </joint>
-    <actuator name="motor_wrist_yaw">
-      <hardwareInterface>EffortJointInterface</hardwareInterface>
-      <mechanicalReduction>1</mechanicalReduction>
-    </actuator>
-  </transmission>
-  <transmission name="trans_wrist_roll">
-    <type>transmission_interface/SimpleTransmission</type>
-    <joint name="wrist_roll_joint">
-      <hardwareInterface>EffortJointInterface</hardwareInterface>
-    </joint>
-    <actuator name="motor_wrist_roll">
-      <hardwareInterface>EffortJointInterface</hardwareInterface>
-      <mechanicalReduction>1</mechanicalReduction>
-    </actuator>
-  </transmission>
+  <xacro:arm_transmission name="shoulder_roll"/>
+  <xacro:arm_transmission name="shoulder_pitch"/>
+  <xacro:arm_transmission name="elbow_pitch"/>
+  <xacro:arm_transmission name="wrist_pitch"/>
+  <xacro:arm_transmission name="wrist_yaw"/>
+  <xacro:arm_transmission name="wrist_roll"/>
 </robot>

Commit message: update description

File: hir_description/urdf/manipulator/manipulator.transmission.xacro (robot description, xacro)
@@ -13,4 +13,5 @@
 	</transmission>
   </xacro:macro>
+<!--
   <transmission name="trans_shoulder_slider">
     <type>transmission_interface/SimpleTransmission</type>
@@ -23,4 +24,5 @@
     </actuator>
   </transmission>
+-->
   <xacro:arm_transmission name="shoulder_roll"/>
   <xacro:arm_transmission name="shoulder_pitch"/>

File: hir_description/urdf/manipulator/manipulator.urdf.xacro (robot description, xacro)
@@ -6,5 +6,5 @@
 	<xacro:include filename="$(find hir_description)/urdf/manipulator/manipulator.transmission.xacro" />
   <!-- joint 0 -->
-  <joint name="shoulder_slider" type="prismatic">
+  <joint name="shoulder_slider" type="fixed">
     <!-- <origin xyz="0.01 0 0.79" rpy="0 0 -1.5707"/> -->
 	<origin xyz="0.01 0 0.9" rpy="0 0 -1.5707" />
