Commit message: increase height

File: hir_description/urdf/manipulator/manipulator.urdf.xacro (robot description, xacro)
@@ -7,5 +7,6 @@
   <!-- joint 0 -->
   <joint name="shoulder_slider" type="prismatic">
-    <origin xyz="0.01 0 0.79" rpy="0 0 -1.5707"/>
+    <!-- <origin xyz="0.01 0 0.79" rpy="0 0 -1.5707"/> -->
+	<origin xyz="0.01 0 0.9" rpy="0 0 -1.5707" />
     <parent link="base_link"/>
     <child link="shoulder_link"/>

Commit message: remove unecessary joint

File: hir_description/urdf/manipulator/manipulator.urdf.xacro (robot description, xacro)
@@ -37,5 +37,5 @@
   </link>
   <!-- joint 1 -->
-  <joint name="shoulder_roll_joint" type="revolute">
+  <joint name="shoulder_roll_joint" type="fixed">
     <origin xyz="0 0.1 0.03" rpy="0 0 0"/>
     <parent link="shoulder_link"/>
@@ -177,5 +177,5 @@
   </link>
   <!--joint 6 + hand -->
-  <joint name="wrist_roll_joint" type="revolute">
+  <joint name="wrist_roll_joint" type="fixed">
     <origin xyz="0 0 -0.05" rpy="0 0 0"/>
     <parent link="wrist_yaw_link"/>
